File: RaspberryPiPCB/PiHat.brd (EAGLE design)
At the start: 65 x 56.5 mm, 19 parts, among them IC1 TPS77030, U1 CAT24C32

Commit message: Final design for manufacturing
Parts:
- removed C1: 10uF, rcl:C1206
- removed C2: 470nF, rcl:C1206
- removed C3: 1uF, rcl:C0603
- removed R11: 47k, rcl:R1206
- removed R3: 3.9K, microbuilder:0805-NO
- removed R9: (no value), rcl:R1206
- removed SJ1: WP, microbuilder:SOLDERJUMPER_CLOSEDWIRE
- removed SL1: (no value), con-amp-quick:07P
- removed SL2: (no value), con-amp-quick:06P
- removed U$4: G2XX3---RHB32, TI_MSP430_v16:RHB32
- removed U1: CAT24C32, microbuilder:SOIC8_150MIL
- added 0.1UF: 0.1uF, rcl:C0603
- added 10UF: 10uF, rcl:C1206
- added 1UF: 1uF, rcl:C0603
- added 470NF: 470nF, rcl:C0603
- added 47K: 47k, rcl:R0603
- added AMT102: (no value), con-lstb-mod:MA06-1
- added DSC6083: DSC6083CI2A-002K000-ND, crystal-geyer_V1_0:3.2X2.5_KXO-V96
- added LED1, LED2: (no value), led:CHIPLED_1206
- added PROGRAM: (no value), con-lstb-mod:MA07-1
- added SV1: (no value), con-lstb-mod:MA08-2
- added U$1: G2XX3---PW28, TI_MSP430_v16:PW28
- R1, R2: value 3.9K -> 300; device microbuilder:0805-NO -> rcl:R0603
- moved IC1 57.0 mm to (6.86, 46.7), turned to 270 degrees
- moved R2 42.8 mm to (13.2, 5.33), turned to 0 degrees
- moved S1 35.7 mm to (35.6, 4.83)
- moved R1 33.9 mm to (20.8, 5.33), turned to 0 degrees
- moved U$2 20.3 mm to (50.9, 2.03)
Connections:
- removed net N$16: R3.1, SJ1.2, U1.7
- removed net N$24: U$4.4
- removed net TA0CLK: U$4.31
- new net INCLK: DSC6083.3, U$1.27
- new net LED0: LED1.A, U$1.10
- new net LED1: LED2.A, U$1.11
- new net N$1: LED1.C, R1.1
- new net N$2: LED2.C, R2.1
- new net N$4: U$1.12
- net 3.3V: no longer R1.2, R2.2, R3.2, U1.8
- net 5.0V: now also 1UF.1; no longer C3.1
- net 5V: now also PROGRAM.6; no longer SL1.6
- net BUTTON: now also 470NF.1, U$1.23; no longer C2.2, R9.2, U$4.3
- net EECLK: no longer R2.1, U1.6
- net EEDATA: no longer R1.1, U1.5
- net GND: now also 0.1UF.2, 10UF.2, 1UF.2, 470NF.2, AMT102.2, DSC6083.2, PROGRAM.7, R1.2, R2.2, SV1.10, SV1.12, SV1.14, SV1.16, SV1.2, SV1.4, SV1.6, SV1.8, U$1.28; no longer C1.2, C2.1, C3.2, SJ1.1, SL1.7, SL2.2, U$4.27, U$4.28, U1.1, U1.2, U1.3, U1.4
- net GPIO16: now also SV1.1, U$1.9; no longer U$4.7
- net GPIO17: now also SV1.3, U$1.8; no longer U$4.6
- net GPIO18: now also SV1.5, U$1.13; no longer U$4.12
- net GPIO19: now also SV1.7, U$1.14; no longer U$4.13
- net GPIO24: now also SV1.9, U$1.15; no longer U$4.14
- net GPIO25: now also SV1.11, U$1.19; no longer U$4.18
- net GPIO26: now also SV1.13, U$1.20; no longer U$4.19
- net GPIO27: now also SV1.15, U$1.21; no longer U$4.20
- net GPIO5: now also U$1.2
- net GPIO6: now also U$1.22
- net MSP_RXD: now also U$1.3; no longer U$4.1
- net MSP_TXD: now also U$1.4; no longer U$4.2
- net N$6: now also AMT102.1; no longer SL2.1
- net QUAD_A: now also AMT102.4, U$1.17; no longer SL2.4, U$4.9
- net QUAD_B: now also AMT102.6, U$1.16; no longer SL2.6, U$4.10
- net QUAD_Z: now also AMT102.3, U$1.18; no longer SL2.3, U$4.11
- net RXD: now also PROGRAM.4; no longer SL1.4
- net SBWTCK: now also PROGRAM.1, U$1.25; no longer SL1.1, U$4.24
- net SBWTDIO: now also 47K.2, PROGRAM.2, U$1.24; no longer R11.2, SL1.2, U$4.23
- net TXD: now also PROGRAM.3; no longer SL1.3
- net VDD: now also 0.1UF.1, 10UF.1, 47K.1, AMT102.5, DSC6083.4, PROGRAM.5, U$1.1; no longer C1.1, R11.1, R9.1, SL1.5, SL2.5, U$4.29, U$4.30
Routing:
- net VDD: track 0.00 -> 108.6 mm, vias 0 -> 5
- net SBWTDIO: track 0.00 -> 60.9 mm
- net GPIO27: track 0.00 -> 59.1 mm, vias 0 -> 1
- net SBWTCK: track 0.00 -> 57.8 mm
- net GPIO16: track 0.00 -> 55.1 mm, vias 0 -> 1
- net GPIO26: track 0.00 -> 54.3 mm, vias 0 -> 1
- net GPIO24: track 0.00 -> 52.8 mm, vias 0 -> 2
- net GPIO19: track 0.00 -> 47.6 mm, vias 0 -> 1
- net GPIO25: track 0.00 -> 43.1 mm
- net GPIO6: track 0.00 -> 43.0 mm
- net MSP_RXD: track 0.00 -> 41.0 mm, vias 0 -> 1
- net MSP_TXD: track 0.00 -> 37.5 mm, vias 0 -> 1
- net GPIO5: track 0.00 -> 34.2 mm, vias 0 -> 2
- net GPIO18: track 0.00 -> 32.2 mm, vias 0 -> 2
- net QUAD_B: track 0.00 -> 30.5 mm
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- added copper zone on layer 1, net GND
- added copper zone on layer 16, net GND
Other:
- board text added: "(c) 2019 sdg"
- board text added: "GND"
- board text added: "GPIO16 GPIO17 GPIO18 GPIO19 GPIO24 GPIO25 GPIO26 GPIO27"
- board text added: "NE"
- board text added: "RNEL Treadmill Tracker+IO [v1.2019]"
- board text added: "SIG"
- board text removed: "WP"
