File: RaspberryPiPCB/PiHat.sch (EAGLE design)
At the start: 18 parts, among them IC1 TPS77030, U1 CAT24C32

Commit message: Final design for manufacturing
Parts:
- removed C1: 10uF, rcl:C-USC1206
- removed C2: 470nF, rcl:C-USC1206
- removed C3: 1uF, rcl:C-USC0603
- removed R11: 47k, rcl:R-US_R1206
- removed R3: 3.9K, microbuilder:RESISTOR0805_NOOUTLINE
- removed R9: (no value), rcl:R-US_R1206
- removed SJ1: WP, microbuilder:SOLDERJUMPER_CLOSED
- removed SL1: (no value), con-amp-quick:M07
- removed SL2: (no value), con-amp-quick:M06
- removed U$4: G2XX3---RHB32, TI_MSP430_v16:G2XX3---RHB32
- removed U1: CAT24C32, microbuilder:EEPROM_I2C_SOIC8_GENERIC
- added 0.1UF: 0.1uF, rcl:C-USC0603
- added 10UF: 10uF, rcl:C-USC1206
- added 1UF: 1uF, rcl:C-USC0603
- added 470NF: 470nF, rcl:C-USC0603
- added 47K: 47k, rcl:R-US_R0603
- added AMT102: (no value), con-lstb-mod:MA06-1
- added DSC6083: DSC6083CI2A-002K000-ND, crystal-geyer_V1_0:KXO-PXO/XO-V96
- added LED1, LED2: (no value), led:LEDCHIPLED_1206
- added PROGRAM: (no value), con-lstb-mod:MA07-1
- added SV1: (no value), con-lstb-mod:MA08-2
- added U$1: G2XX3---PW28, TI_MSP430_v16:G2XX3---PW28
- R1, R2: value 3.9K -> 300; device microbuilder:RESISTOR0805_NOOUTLINE -> rcl:R-US_R0603
Connections:
- removed net N$16: R3.1, SJ1.2, U1.WP
- removed net N$24: U$4.4
- removed net TA0CLK: U$4.31
- new net INCLK: DSC6083.OUT, U$1.27
- new net LED0: LED1.A, U$1.10
- new net LED1: LED2.A, U$1.11
- new net N$1: LED1.C, R1.1
- new net N$2: LED2.C, R2.1
- new net N$4: U$1.12
- net 3.3V: no longer R1.2, R2.2, R3.2, U1.VCC
- net 5.0V: now also 1UF.1; no longer C3.1
- net 5V: now also PROGRAM.6; no longer SL1.6
- net BUTTON: now also 470NF.1, U$1.23; no longer C2.2, R9.2, U$4.3
- net EECLK: no longer R2.1, U1.SCL
- net EEDATA: no longer R1.1, U1.SDA
- net GND: now also 0.1UF.2, 10UF.2, 1UF.2, 470NF.2, AMT102.2, DSC6083.GND, PROGRAM.7, R1.2, R2.2, SV1.10, SV1.12, SV1.14, SV1.16, SV1.2, SV1.4, SV1.6, SV1.8, U$1.28; no longer C1.2, C2.1, C3.2, SJ1.1, SL1.7, SL2.2, U$4.27, U$4.28, U1.A0, U1.A1, U1.A2, U1.GND
- net GPIO16: now also SV1.1, U$1.9; no longer U$4.7
- net GPIO17: now also SV1.3, U$1.8; no longer U$4.6
- net GPIO18: now also SV1.5, U$1.13; no longer U$4.12
- net GPIO19: now also SV1.7, U$1.14; no longer U$4.13
- net GPIO24: now also SV1.9, U$1.15; no longer U$4.14
- net GPIO25: now also SV1.11, U$1.19; no longer U$4.18
- net GPIO26: now also SV1.13, U$1.20; no longer U$4.19
- net GPIO27: now also SV1.15, U$1.21; no longer U$4.20
- net GPIO5: now also U$1.2
- net GPIO6: now also U$1.22
- net MSP_RXD: now also U$1.3; no longer U$4.1
- net MSP_TXD: now also U$1.4; no longer U$4.2
- net N$6: now also AMT102.1; no longer SL2.1
- net QUAD_A: now also AMT102.4, U$1.17; no longer SL2.4, U$4.9
- net QUAD_B: now also AMT102.6, U$1.16; no longer SL2.6, U$4.10
- net QUAD_Z: now also AMT102.3, U$1.18; no longer SL2.3, U$4.11
- net RXD: now also PROGRAM.4; no longer SL1.4
- net SBWTCK: now also PROGRAM.1, U$1.25; no longer SL1.1, U$4.24
- net SBWTDIO: now also 47K.2, PROGRAM.2, U$1.24; no longer R11.2, SL1.2, U$4.23
- net TXD: now also PROGRAM.3; no longer SL1.3
- net VDD: now also 0.1UF.1, 10UF.1, 47K.1, AMT102.5, DSC6083.VDD, PROGRAM.5, U$1.1; no longer C1.1, R11.1, R9.1, SL1.5, SL2.5, U$4.29, U$4.30
