File: PCBs/PiHat.brd (EAGLE design)
At the start: 65 x 56.5 mm, 33 parts, among them U1 TLV70036DDCTDDC5-L, U2 FT230

Commit message: Updated interface PCB to have proper silkscreen and added manufacturing files
Parts:
- S1: value MOMENTARY-SWITCH-SPST-PTH-6.0MM -> (none)
Other:
- board text added: "*"
- board text added: "RNEL Treadmill Tracker+IO [v3.2019]"
- board text removed: "RNEL Treadmill Tracker+IO [v1.2019]"
Changed lines of the file:
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@@
 Treadmill
 Tracker+IO
-[v1.2019]</text>
+[v3.2019]</text>
 <text x="4.826" y="8.89" size="0.8128" layer="22" font="vector" ratio="16" rot="MR90" align="center-left">(c) 2019
 sdg</text>
@@
 <text x="11.938" y="6.604" size="1.27" layer="21" font="vector" ratio="16">PWR</text>
 <text x="18.034" y="6.604" size="1.27" layer="21" font="vector" ratio="16">STATUS</text>
+<text x="21.59" y="20.574" size="1.016" layer="21" font="vector" ratio="20" rot="R180">*</text>
 </plain>
 <attributes>
@@
 </element>
 <element name="U$2" library="microbuilder" package="PIHATLOGO" value="" x="45.847" y="39.878" smashed="yes"/>
-<element name="S1" library="SparkFun-Switches" package="TACTILE_SWITCH_PTH_6.0MM" value="MOMENTARY-SWITCH-SPST-PTH-6.0MM" x="35.56" y="4.826" smashed="yes">
+<element name="S1" library="SparkFun-Switches" package="TACTILE_SWITCH_PTH_6.0MM" value="" x="35.56" y="4.826" smashed="yes">
 <attribute name="PROD_ID" value=" SWCH-08441" x="31.115" y="14.732" size="1.778" layer="27" display="off"/>
 <attribute name="SF_SKU" value="COM-00097" x="31.115" y="14.732" size="1.778" layer="27" display="off"/>
@@
 <element name="DSC6083" library="crystal-geyer_V1_0" library_urn="urn:adsk.eagle:library:203" package="3.2X2.5_KXO-V96" package3d_urn="urn:adsk.eagle:package:11941/1" value="2KHZ" x="19.304" y="22.098" smashed="yes" rot="R90">
 <attribute name="NAME" x="22.628" y="25.478" size="1.016" layer="25" font="vector" ratio="16" rot="R180"/>
-<attribute name="VALUE" x="22.458" y="19.536" size="1.016" layer="27" font="vector" ratio="16" rot="R90"/>
+<attribute name="VALUE" x="21.358" y="19.664" size="1.016" layer="27" font="vector" ratio="16" rot="R180"/>
 </element>
 <element name="C" library="rcl" library_urn="urn:adsk.eagle:library:334" package="C0603" package3d_urn="urn:adsk.eagle:package:23616/2" value="0.1uF" x="16.51" y="20.066" smashed="yes" rot="R270">
 <attribute name="SPICEPREFIX" value="C" x="16.51" y="20.066" size="1.778" layer="27" rot="R270" display="off"/>
-<attribute name="VALUE" x="15.875" y="18.669" size="1.27" layer="27" font="vector" ratio="16" rot="R270"/>
+<attribute name="VALUE" x="15.875" y="18.669" size="1.016" layer="27" font="vector" ratio="15" rot="R270"/>
 </element>
 <element name="470NF" library="rcl" library_urn="urn:adsk.eagle:library:334" package="C0603" package3d_urn="urn:adsk.eagle:package:23616/2" value="470nF" x="28.956" y="4.572" smashed="yes" rot="R90">
@@
 </element>
 <element name="U$1" library="TI_MSP430_v16" package="PW28" value="MSP430" x="28.956" y="17.526" smashed="yes" rot="R270">
-<attribute name="VALUE" x="27.3479" y="20.5051" size="1.016" layer="27" font="vector" ratio="16" rot="R270"/>
+<attribute name="VALUE" x="27.3479" y="20.5051" size="1.016" layer="27" font="vector" ratio="15" rot="R270"/>
 </element>
 <element name="LED1" library="led" library_urn="urn:adsk.eagle:library:259" package="CHIPLED_1206" package3d_urn="urn:adsk.eagle:package:15823/2" value="" x="21.59" y="2.54" smashed="yes" rot="R90">
@@
 <element name="R1" library="rcl" library_urn="urn:adsk.eagle:library:334" package="R0603" package3d_urn="urn:adsk.eagle:package:23555/3" value="R" x="20.828" y="5.334" smashed="yes">
 <attribute name="SPICEPREFIX" value="R" x="20.828" y="5.334" size="1.778" layer="27" display="off"/>
-<attribute name="VALUE" x="18.669" y="4.699" size="1.27" layer="27" rot="R90"/>
 </element>
 <element name="R2" library="rcl" library_urn="urn:adsk.eagle:library:334" package="R0603" package3d_urn="urn:adsk.eagle:package:23555/3" value="R" x="13.208" y="5.334" smashed="yes">
 <attribute name="SPICEPREFIX" value="R" x="13.208" y="5.334" size="1.778" layer="27" display="off"/>
-<attribute name="VALUE" x="11.049" y="4.445" size="1.27" layer="27" rot="R90"/>
 </element>
 <element name="SV1" library="con-lstb-mod" package="MA08-2" package3d_urn="urn:adsk.eagle:package:8335/1" value="" x="30.48" y="40.64" smashed="yes">
@@
 <element name="USB1" library="microftx" package="FCI-10118193-0001LF" value="MICRO-USB-FCI-10118193" x="52.578" y="0" smashed="yes"/>
 <element name="R3" library="resistor" library_urn="urn:adsk.eagle:library:348" package="R0603" package3d_urn="urn:adsk.eagle:package:26057/1" value="27R" x="51.816" y="8.128" smashed="yes" rot="R90">
-<attribute name="VALUE" x="52.197" y="9.779" size="1.016" layer="27" font="vector" ratio="20" rot="R90"/>
+<attribute name="VALUE" x="52.197" y="9.779" size="1.016" layer="27" font="vector" ratio="15" rot="R90"/>
 </element>
 <element name="R4" library="resistor" library_urn="urn:adsk.eagle:library:348" package="R0603" package3d_urn="urn:adsk.eagle:package:26057/1" value="27R" x="55.88" y="8.128" smashed="yes" rot="R90">
-<attribute name="VALUE" x="56.261" y="9.779" size="1.016" layer="27" font="vector" ratio="20" rot="R90"/>
+<attribute name="VALUE" x="56.261" y="9.779" size="1.016" layer="27" font="vector" ratio="15" rot="R90"/>
 </element>
 <element name="FERRITE" library="rcl" library_urn="urn:adsk.eagle:library:334" package="R0805" package3d_urn="urn:adsk.eagle:package:23553/2" value="" x="49.784" y="8.128" smashed="yes" rot="R90">
+<attribute name="NAME" x="50.292" y="10.033" size="0.889" layer="25" font="vector" rot="R90"/>
 <attribute name="SPICEPREFIX" value="R" x="49.784" y="8.128" size="1.778" layer="27" rot="R90" display="off"/>
 <attribute name="VALUE" x="52.324" y="7.493" size="1.27" layer="27" rot="R90"/>
 </element>
 <element name="C3" library="resistor" library_urn="urn:adsk.eagle:library:348" package="C0603" package3d_urn="urn:adsk.eagle:package:26138/1" value="10nF" x="47.498" y="8.128" smashed="yes" rot="R90">
-<attribute name="VALUE" x="47.879" y="10.287" size="1.016" layer="27" font="vector" ratio="20" rot="R90"/>
+<attribute name="VALUE" x="47.879" y="10.287" size="1.016" layer="27" font="vector" ratio="15" rot="R90"/>
 </element>
 <element name="C4" library="resistor" library_urn="urn:adsk.eagle:library:348" package="C0603" package3d_urn="urn:adsk.eagle:package:26138/1" value="100nF" x="48.006" y="19.304" smashed="yes" rot="R90">
-<attribute name="VALUE" x="48.133" y="21.209" size="1.016" layer="27" font="vector" ratio="20" rot="R90"/>
+<attribute name="VALUE" x="48.133" y="21.209" size="1.016" layer="27" font="vector" ratio="15" rot="R90"/>
 </element>
 <element name="C5" library="resistor" library_urn="urn:adsk.eagle:library:348" package="C0603" package3d_urn="urn:adsk.eagle:package:26138/1" value="47pF" x="53.848" y="8.128" smashed="yes" rot="R90">
-<attribute name="VALUE" x="54.229" y="9.779" size="1.016" layer="27" font="vector" ratio="20" rot="R90"/>
+<attribute name="VALUE" x="54.229" y="9.779" size="1.016" layer="27" font="vector" ratio="15" rot="R90"/>
 </element>
 <element name="C6" library="resistor" library_urn="urn:adsk.eagle:library:348" package="C0603" package3d_urn="urn:adsk.eagle:package:26138/1" value="47pF" x="57.912" y="8.128" smashed="yes" rot="R90">
-<attribute name="VALUE" x="58.293" y="9.779" size="1.016" layer="27" font="vector" ratio="20" rot="R90"/>
+<attribute name="VALUE" x="58.293" y="9.779" size="1.016" layer="27" font="vector" ratio="15" rot="R90"/>
 </element>
 <element name="RX" library="led" library_urn="urn:adsk.eagle:library:259" package="CHIPLED_1206" package3d_urn="urn:adsk.eagle:package:15823/2" value="" x="60.96" y="16.51" smashed="yes" rot="R270">
